File: vco/vco.kicad_pcb (KiCad board)
At the start: 2 copper layers, 70 x 100 mm, 34 parts, among them J1 Conn_01x02_Socket, J2 Conn_01x02_Socket, J3 Conn_01x02_Socket, J4 Conn_01x02_Socket, J5 Conn_01x03_Socket, J6 Conn_01x03_Socket, Q1 BC548C, Q2 BC558, U1 40106, U2 TL074

Commit message: increase track width and clearance + reroute
Routing:
- net -12V: track 108.0 -> 106.1 mm
- net GND: track 223.9 -> 225.8 mm
- net Net-(D1-K): track 58.8 -> 60.7 mm, vias 0 -> 1
- net +12V: track 136.2 -> 137.2 mm
- net Net-(J5-Pin_2): track 51.6 -> 52.6 mm
- net Net-(D1-A): track 10.7 -> 11.6 mm
