File: vco/vco.kicad_pcb (KiCad board)
At the start: 2 copper layers, 70 x 100 mm, 34 parts, among them J1 Conn_01x02_Socket, J2 Conn_01x02_Socket, J3 Conn_01x02_Socket, J4 Conn_01x02_Socket, J5 Conn_01x03_Socket, J6 Conn_01x03_Socket, Q1 BC548C, Q2 BC558, U1 40106, U2 TL074

Commit message: fix missing resistor add link to yt add vco bom
Parts:
- moved J4 7.55 mm to (123.2, 99.0)
- moved J5 7.55 mm to (123.2, 111.7)
- moved R11 7.55 mm to (166.9, 76.1)
- moved R12 7.55 mm to (156.8, 80.7)
- moved R15 7.55 mm to (143.5, 103.6)
- moved R16 7.55 mm to (118.7, 81.2)
- moved R17 7.55 mm to (118.7, 85.3)
- moved R2 7.55 mm to (153.7, 63.9)
- moved R9 7.55 mm to (131.9, 76.6)
- moved RV4 7.55 mm to (118.7, 71.1)
- moved U2 7.55 mm to (145.1, 76.6)
- moved C2 7.55 mm to (138.0, 68.8)
- moved J2 7.55 mm to (172.5, 78.2)
- moved J3 7.55 mm to (176.6, 99.5)
- moved R1 7.55 mm to (157.3, 47.7)
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