File: vco/vco.kicad_sch (KiCad schematic)
At the start: 34 parts, among them J1 Conn_01x02_Socket, J2 Conn_01x02_Socket, J3 Conn_01x02_Socket, J4 Conn_01x02_Socket, J5 Conn_01x03_Socket, J6 Conn_01x03_Socket, Q1 BC548C, Q2 BC558, U1 40106, U2 TL074

Commit message: fix missing resistor add link to yt add vco bom
Parts:
- added R18: 100k, Resistor_THT:R_Axial_DIN0207_L6.3mm_D2.5mm_P10.16mm_Horizontal, symbol Device:R
Connections:
- net at R16.2, R17.2, U2.6 (-): now also R18.2; no longer J5.2 (Pin_2)
- new net: J5.2 (Pin_2), R18.1
Changed lines of the file:
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@@
   (no_connect (at 276.352 64.516))
   (no_connect (at 273.812 52.324))
+  (wire (pts (xy 123.952 154.178) (xy 145.7367 154.178))
+    (stroke (width 0) (type default))
+  )
   (wire (pts (xy 125.984 77.724) (xy 125.984 87.1551))
     (stroke (width 0) (type default))
@@
   )
   (wire (pts (xy 85.852 104.14) (xy 85.852 110.236))
-    (stroke (width 0) (type default))
-  )
-  (wire (pts (xy 116.332 154.178) (xy 145.7367 154.178))
     (stroke (width 0) (type default))
   )
@@
         )
       )
+    )
+  )
+  (symbol (lib_id "Device:R") (at 120.142 154.178 90) (unit 1)
+    (in_bom yes) (on_board yes) (dnp no) (fields_autoplaced)
+    (property "Reference" "R18" (at 120.142 148.59 90)
+      (effects (font (size 1.27 1.27)))
+    )
+    (property "Value" "100k" (at 120.142 151.13 90)
+      (effects (font (size 1.27 1.27)))
+    )
+    (property "Footprint" "Resistor_THT:R_Axial_DIN0207_L6.3mm_D2.5mm_P10.16mm_Horizontal" (at 120.142 155.956 90)
+      (effects (font (size 1.27 1.27)) hide)
+    )
+    (property "Datasheet" "~" (at 120.142 154.178 0)
+      (effects (font (size 1.27 1.27)) hide)
+    )
+    (pin "1")
+    (pin "2")
+    (instances
+      (project "vco"
+        (path "/7ad23056-9872-4bcb-9d54-52246d8eb9ad"
+          (reference "R18") (unit 1)
+        )
+      )
