File: env/env.kicad_sch (KiCad schematic)
At the start: 35 parts, among them J1 Conn_01x02_Socket, J2 Conn_01x03_Socket, J3 Conn_01x02_Socket, J4 Conn_01x02_Socket, Q1 BC548C, SW1 SW_SPDT, U1 TL074, U2 TL074

Commit message: turn vca to dual vca add mounting holes
Parts:
- added H1, H2, H3, H4: MountingHole, MountingHole:MountingHole_2.1mm, symbol Mechanical:MountingHole
Changed lines of the file:
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@@
+    )
+  )
+  (symbol (lib_id "Mechanical:MountingHole") (at 90.17 29.972 0) (unit 1)
+    (in_bom yes) (on_board yes) (dnp no) (fields_autoplaced)
+    (property "Reference" "H2" (at 93.599 28.702 0)
+      (effects (font (size 1.27 1.27)) (justify left))
+    )
+    (property "Value" "MountingHole" (at 93.599 31.242 0)
+      (effects (font (size 1.27 1.27)) (justify left))
+    )
+    (property "Footprint" "MountingHole:MountingHole_2.1mm" (at 90.17 29.972 0)
+      (effects (font (size 1.27 1.27)) hide)
+    )
+    (property "Datasheet" "~" (at 90.17 29.972 0)
+      (effects (font (size 1.27 1.27)) hide)
+    )
+    (instances
+      (project "env"
+        (path "/184ccf12-cca4-4023-8353-c346776e6856"
+          (reference "H2") (unit 1)
+        )
+      )
     )
   )
@@
     )
   )
+  (symbol (lib_id "Mechanical:MountingHole") (at 93.218 42.037 0) (unit 1)
+    (in_bom yes) (on_board yes) (dnp no) (fields_autoplaced)
+    (property "Reference" "H4" (at 96.647 40.767 0)
+      (effects (font (size 1.27 1.27)) (justify left))
+    )
+    (property "Value" "MountingHole" (at 96.647 43.307 0)
+      (effects (font (size 1.27 1.27)) (justify left))
+    )
+    (property "Footprint" "MountingHole:MountingHole_2.1mm" (at 93.218 42.037 0)
+      (effects (font (size 1.27 1.27)) hide)
+    )
+    (property "Datasheet" "~" (at 93.218 42.037 0)
+      (effects (font (size 1.27 1.27)) hide)
+    )
+    (instances
+      (project "env"
+        (path "/184ccf12-cca4-4023-8353-c346776e6856"
+          (reference "H4") (unit 1)
+        )
+      )
+    )
+  )
   (symbol (lib_id "power:GND") (at 60.96 92.71 0) (unit 1)
     (in_bom yes) (on_board yes) (dnp no) (fields_autoplaced)
@@
         (path "/184ccf12-cca4-4023-8353-c346776e6856"
           (reference "#PWR016") (unit 1)
+        )
+      )
+    )
+  )
+  (symbol (lib_id "Mechanical:MountingHole") (at 89.281 24.638 0) (unit 1)
+    (in_bom yes) (on_board yes) (dnp no) (fields_autoplaced)
+    (property "Reference" "H1" (at 92.71 23.368 0)
+      (effects (font (size 1.27 1.27)) (justify left))
+    )
+    (property "Value" "MountingHole" (at 92.71 25.908 0)
+      (effects (font (size 1.27 1.27)) (justify left))
+    )
+    (property "Footprint" "MountingHole:MountingHole_2.1mm" (at 89.281 24.638 0)
+      (effects (font (size 1.27 1.27)) hide)
+    )
+    (property "Datasheet" "~" (at 89.281 24.638 0)
+      (effects (font (size 1.27 1.27)) hide)
+    )
+    (instances
+      (project "env"
+        (path "/184ccf12-cca4-4023-8353-c346776e6856"
+          (reference "H1") (unit 1)
         )
       )
@@
         )
       )
+    )
+  )
+  (symbol (lib_id "Mechanical:MountingHole") (at 91.313 35.814 0) (unit 1)
+    (in_bom yes) (on_board yes) (dnp no) (fields_autoplaced)
+    (property "Reference" "H3" (at 94.742 34.544 0)
+      (effects (font (size 1.27 1.27)) (justify left))
+    )
+    (property "Value" "MountingHole" (at 94.742 37.084 0)
+      (effects (font (size 1.27 1.27)) (justify left))
+    )
+    (property "Footprint" "MountingHole:MountingHole_2.1mm" (at 91.313 35.814 0)
+      (effects (font (size 1.27 1.27)) hide)
+    )
+    (property "Datasheet" "~" (at 91.313 35.814 0)
+      (effects (font (size 1.27 1.27)) hide)
+    )
+    (instances
+      (project "env"
+        (path "/184ccf12-cca4-4023-8353-c346776e6856"
+          (reference "H3") (unit 1)
+        )
+      )

Commit message: use custom footprints with bigger pads
Parts:
- C1, C2: footprint Capacitor_THT:C_Disc_D4.3mm_W1.9mm_P5.00mm -> my_tht_cap
- D1, D2, D3, D4, D5, D6: footprint Diode_THT:D_DO-35_SOD27_P7.62mm_Horizontal -> my_library:my_tht_diode
- R1, R10, R11, R12, R13, R14, R15, R2, R3, R4, R5, R6, R7, R8, R9: footprint Resistor_THT:R_Axial_DIN0204_L3.6mm_D1.6mm_P7.62mm_Horizontal -> my_library:my_tht_r
Changed lines of the file:
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@@
       (effects (font (size 1.27 1.27)))
     )
-    (property "Footprint" "Resistor_THT:R_Axial_DIN0204_L3.6mm_D1.6mm_P7.62mm_Horizontal" (at 211.836 72.1156 90)
+    (property "Footprint" "my_library:my_tht_r" (at 211.836 72.1156 90)
       (effects (font (size 1.27 1.27)) hide)
     )
@@
       (effects (font (size 1.27 1.27)) (justify left))
     )
-    (property "Footprint" "Diode_THT:D_DO-35_SOD27_P7.62mm_Horizontal" (at 50.8 88.138 0)
+    (property "Footprint" "my_library:my_tht_diode" (at 50.8 88.138 0)
       (effects (font (size 1.27 1.27)) hide)
     )
@@
       (effects (font (size 1.27 1.27)))
     )
-    (property "Footprint" "Resistor_THT:R_Axial_DIN0204_L3.6mm_D1.6mm_P7.62mm_Horizontal" (at 214.63 95.758 90)
+    (property "Footprint" "my_library:my_tht_r" (at 214.63 95.758 90)
       (effects (font (size 1.27 1.27)) hide)
     )
@@
       (effects (font (size 1.27 1.27)))
     )
-    (property "Footprint" "Resistor_THT:R_Axial_DIN0204_L3.6mm_D1.6mm_P7.62mm_Horizontal" (at 160.274 105.2666 90)
+    (property "Footprint" "my_library:my_tht_r" (at 160.274 105.2666 90)
       (effects (font (size 1.27 1.27)) hide)
     )
@@
       (effects (font (size 1.27 1.27)) (justify right))
     )
-    (property "Footprint" "Capacitor_THT:C_Disc_D4.3mm_W1.9mm_P5.00mm" (at 177.6915 82.042 0)
+    (property "Footprint" "my_tht_cap" (at 177.6915 82.042 0)
       (effects (font (size 1.27 1.27)) hide)
     )
@@
       (effects (font (size 1.27 1.27)))
     )
-    (property "Footprint" "Resistor_THT:R_Axial_DIN0204_L3.6mm_D1.6mm_P7.62mm_Horizontal" (at 226.06 102.616 90)
+    (property "Footprint" "my_library:my_tht_r" (at 226.06 102.616 90)
       (effects (font (size 1.27 1.27)) hide)
     )
@@
       (effects (font (size 1.27 1.27)))
     )
-    (property "Footprint" "Capacitor_THT:C_Disc_D4.3mm_W1.9mm_P5.00mm" (at 50.8 83.3628 0)
+    (property "Footprint" "my_tht_cap" (at 50.8 83.3628 0)
       (effects (font (size 1.27 1.27)) hide)
     )
@@
       (effects (font (size 1.27 1.27)))
     )
-    (property "Footprint" "Diode_THT:D_DO-35_SOD27_P7.62mm_Horizontal" (at 93.472 84.582 0)
+    (property "Footprint" "my_library:my_tht_diode" (at 93.472 84.582 0)
       (effects (font (size 1.27 1.27)) hide)
     )
@@
       (effects (font (size 1.27 1.27)) (justify left))
     )
-    (property "Footprint" "Resistor_THT:R_Axial_DIN0204_L3.6mm_D1.6mm_P7.62mm_Horizontal" (at 87.884 101.6 90)
+    (property "Footprint" "my_library:my_tht_r" (at 87.884 101.6 90)
       (effects (font (size 1.27 1.27)) hide)
     )
@@
       (effects (font (size 1.27 1.27)) (justify left))
     )
-    (property "Footprint" "Resistor_THT:R_Axial_DIN0204_L3.6mm_D1.6mm_P7.62mm_Horizontal" (at 96.012 113.538 90)
+    (property "Footprint" "my_library:my_tht_r" (at 96.012 113.538 90)
       (effects (font (size 1.27 1.27)) hide)
     )
@@
       (effects (font (size 1.27 1.27)) (justify left))
     )
-    (property "Footprint" "Resistor_THT:R_Axial_DIN0204_L3.6mm_D1.6mm_P7.62mm_Horizontal" (at 194.31 109.22 90)
+    (property "Footprint" "my_library:my_tht_r" (at 194.31 109.22 90)
       (effects (font (size 1.27 1.27)) hide)
     )
@@
       (effects (font (size 1.27 1.27)))
     )
-    (property "Footprint" "Resistor_THT:R_Axial_DIN0204_L3.6mm_D1.6mm_P7.62mm_Horizontal" (at 167.894 118.11 90)
+    (property "Footprint" "my_library:my_tht_r" (at 167.894 118.11 90)
       (effects (font (size 1.27 1.27)) hide)
     )
@@
       (effects (font (size 1.27 1.27)))
     )
-    (property "Footprint" "Diode_THT:D_DO-35_SOD27_P7.62mm_Horizontal" (at 159.004 71.12 0)
+    (property "Footprint" "my_library:my_tht_diode" (at 159.004 71.12 0)
       (effects (font (size 1.27 1.27)) hide)
     )
@@
       (effects (font (size 1.27 1.27)))
     )
-    (property "Footprint" "Diode_THT:D_DO-35_SOD27_P7.62mm_Horizontal" (at 161.036 85.852 0)
+    (property "Footprint" "my_library:my_tht_diode" (at 161.036 85.852 0)
       (effects (font (size 1.27 1.27)) hide)
     )
@@
       (effects (font (size 1.27 1.27)) (justify right))
     )
-    (property "Footprint" "Resistor_THT:R_Axial_DIN0204_L3.6mm_D1.6mm_P7.62mm_Horizontal" (at 207.264 89.408 90)
+    (property "Footprint" "my_library:my_tht_r" (at 207.264 89.408 90)
       (effects (font (size 1.27 1.27)) hide)
     )
@@
       (effects (font (size 1.27 1.27)) (justify right))
     )
-    (property "Footprint" "Resistor_THT:R_Axial_DIN0204_L3.6mm_D1.6mm_P7.62mm_Horizontal" (at 197.866 116.84 90)
+    (property "Footprint" "my_library:my_tht_r" (at 197.866 116.84 90)
       (effects (font (size 1.27 1.27)) hide)
     )
@@
       (effects (font (size 1.27 1.27)) (justify left))
     )
-    (property "Footprint" "Resistor_THT:R_Axial_DIN0204_L3.6mm_D1.6mm_P7.62mm_Horizontal" (at 87.884 93.98 90)
+    (property "Footprint" "my_library:my_tht_r" (at 87.884 93.98 90)
       (effects (font (size 1.27 1.27)) hide)
     )
@@
       (effects (font (size 1.27 1.27)))
     )
-    (property "Footprint" "Resistor_THT:R_Axial_DIN0204_L3.6mm_D1.6mm_P7.62mm_Horizontal" (at 148.844 81.026 90)
+    (property "Footprint" "my_library:my_tht_r" (at 148.844 81.026 90)
       (effects (font (size 1.27 1.27)) hide)
     )
@@
       (effects (font (size 1.27 1.27)) (justify left))
     )
-    (property "Footprint" "Resistor_THT:R_Axial_DIN0204_L3.6mm_D1.6mm_P7.62mm_Horizontal" (at 59.182 88.9 90)
+    (property "Footprint" "my_library:my_tht_r" (at 59.182 88.9 90)
       (effects (font (size 1.27 1.27)) hide)
     )
@@
       (effects (font (size 1.27 1.27)) (justify right))
     )
-    (property "Footprint" "Resistor_THT:R_Axial_DIN0204_L3.6mm_D1.6mm_P7.62mm_Horizontal" (at 143.002 122.682 90)
+    (property "Footprint" "my_library:my_tht_r" (at 143.002 122.682 90)
       (effects (font (size 1.27 1.27)) hide)
     )
@@
       (effects (font (size 1.27 1.27)))
     )
-    (property "Footprint" "Diode_THT:D_DO-35_SOD27_P7.62mm_Horizontal" (at 145.034 118.872 0)
+    (property "Footprint" "my_library:my_tht_diode" (at 145.034 118.872 0)
       (effects (font (size 1.27 1.27)) hide)
     )
@@
       (effects (font (size 1.27 1.27)))
     )
-    (property "Footprint" "Diode_THT:D_DO-35_SOD27_P7.62mm_Horizontal" (at 90.17 121.158 0)
+    (property "Footprint" "my_library:my_tht_diode" (at 90.17 121.158 0)
       (effects (font (size 1.27 1.27)) hide)
     )
@@
       (effects (font (size 1.27 1.27)) (justify right))
     )
-    (property "Footprint" "Resistor_THT:R_Axial_DIN0204_L3.6mm_D1.6mm_P7.62mm_Horizontal" (at 165.862 102.108 90)
-      (effects (font (size 1.27 1.27)) hide)
-    )
+    (property "Footprint" "my_library:my_tht_r" (at 165.862 102.108 90)
+      (effects (font (size 1.27 1.27)) hide)
+    )

Commit message: update almost all other footprints to fatty pads
Parts:
- Q1: footprint BC548C:TO92250P510H770-3 -> my_library:my_bc548
Changed lines of the file:
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@@
       (effects (font (size 1.27 1.27)) (justify left))
     )
-    (property "Footprint" "BC548C:TO92250P510H770-3" (at 233.68 91.186 0)
+    (property "Footprint" "my_library:my_bc548" (at 233.68 91.186 0)
       (effects (font (size 1.27 1.27)) (justify bottom) hide)
     )

Commit message: FRIENDSHIP ENDED WITH PACKAGE_DIP. added a keep-out on F.cu for dip14
Parts:
- U1, U2: footprint my_library:my_dip14 -> my_library:my_dip14_no_f_pads
Changed lines of the file:
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@@
       (effects (font (size 1.27 1.27)))
     )
-    (property "Footprint" "my_library:my_dip14" (at 77.47 123.698 0)
+    (property "Footprint" "my_library:my_dip14_no_f_pads" (at 77.47 123.698 0)
       (effects (font (size 1.27 1.27)) hide)
     )
@@
       (effects (font (size 1.27 1.27)))
     )
-    (property "Footprint" "my_library:my_dip14" (at 136.144 85.344 0)
+    (property "Footprint" "my_library:my_dip14_no_f_pads" (at 136.144 85.344 0)
       (effects (font (size 1.27 1.27)) hide)
     )
@@
       (effects (font (size 1.27 1.27)))
     )
-    (property "Footprint" "my_library:my_dip14" (at 157.734 116.332 0)
+    (property "Footprint" "my_library:my_dip14_no_f_pads" (at 157.734 116.332 0)
       (effects (font (size 1.27 1.27)) hide)
     )
@@
       (effects (font (size 1.27 1.27)))
     )
-    (property "Footprint" "my_library:my_dip14" (at 262.89 109.982 0)
+    (property "Footprint" "my_library:my_dip14_no_f_pads" (at 262.89 109.982 0)
       (effects (font (size 1.27 1.27)) hide)
     )
@@
       (effects (font (size 1.27 1.27)))
     )
-    (property "Footprint" "my_library:my_dip14" (at 213.36 106.934 0)
+    (property "Footprint" "my_library:my_dip14_no_f_pads" (at 213.36 106.934 0)
       (effects (font (size 1.27 1.27)) hide)
     )
@@
       (effects (font (size 1.27 1.27)) (justify left))
     )
-    (property "Footprint" "my_library:my_dip14" (at 274.828 81.788 0)
+    (property "Footprint" "my_library:my_dip14_no_f_pads" (at 274.828 81.788 0)
       (effects (font (size 1.27 1.27)) hide)
     )
@@
       (effects (font (size 1.27 1.27)))
     )
-    (property "Footprint" "my_library:my_dip14" (at 264.16 127.508 0)
+    (property "Footprint" "my_library:my_dip14_no_f_pads" (at 264.16 127.508 0)
       (effects (font (size 1.27 1.27)) hide)
     )
@@
       (effects (font (size 1.27 1.27)))
     )
-    (property "Footprint" "my_library:my_dip14" (at 80.772 82.042 0)
+    (property "Footprint" "my_library:my_dip14_no_f_pads" (at 80.772 82.042 0)
       (effects (font (size 1.27 1.27)) hide)
     )
@@
       (effects (font (size 1.27 1.27)))
     )
-    (property "Footprint" "my_library:my_dip14" (at 199.136 76.2 0)
+    (property "Footprint" "my_library:my_dip14_no_f_pads" (at 199.136 76.2 0)
       (effects (font (size 1.27 1.27)) hide)
     )
@@
       (effects (font (size 1.27 1.27)) (justify left))
     )
-    (property "Footprint" "my_library:my_dip14" (at 265.43 85.344 0)
-      (effects (font (size 1.27 1.27)) hide)
-    )
+    (property "Footprint" "my_library:my_dip14_no_f_pads" (at 265.43 85.344 0)
+      (effects (font (size 1.27 1.27)) hide)
+    )
